Commit message: minor changes at xacro file

File: src/third-party/mycobot-ros2/mycobot_description/urdf/mech/axtbot_arm.urdf.xacro (robot description, xacro)
@@ -158,5 +158,5 @@
       <parent link="${prefix}link2"/>
       <child link="${prefix}link3"/>
-      <origin xyz="0 0 -0.001" rpy="${pi/2} ${-pi/2} ${pi/2}"/>
+      <origin xyz="0 0 -0.001" rpy="0 ${-pi/2} ${pi/2}"/>
       <dynamics damping="${joint_damping}" friction="${joint_friction}"/>
     </joint>

Commit message: pasando los link de tipo revolute a fixed

File: src/third-party/mycobot-ros2/mycobot_description/urdf/mech/axtbot_arm.urdf.xacro (robot description, xacro)
@@ -145,5 +145,5 @@
       <xacro:insert_block name="origin"/>
     </joint>
-    <joint name="${prefix}link1_to_${prefix}link2" type="revolute">
+    <joint name="${prefix}link1_to_${prefix}link2" type="fixed">
       <axis xyz="0 0 1"/>
       <limit effort="${joint_effort}" lower="-2.9321" upper="2.9321" velocity="${joint_velocity}"/>
@@ -153,5 +153,5 @@
       <dynamics damping="${joint_damping}" friction="${joint_friction}"/>
     </joint>
-    <joint name="${prefix}link2_to_${prefix}link3" type="revolute">
+    <joint name="${prefix}link2_to_${prefix}link3" type="fixed">
       <axis xyz="0 0 1"/>
       <limit effort="${joint_effort}" lower="-2.3561" upper="2.3561" velocity="${joint_velocity}"/>
@@ -161,5 +161,5 @@
       <dynamics damping="${joint_damping}" friction="${joint_friction}"/>
     </joint>
-    <joint name="${prefix}link3_to_${prefix}link4" type="revolute">
+    <joint name="${prefix}link3_to_${prefix}link4" type="fixed">
       <axis xyz="0 0 1"/>
       <limit effort="${joint_effort}" lower="-2.5307" upper="2.5307" velocity="${joint_velocity}"/>
@@ -169,5 +169,5 @@
       <dynamics damping="${joint_damping}" friction="${joint_friction}"/>
     </joint>
-    <joint name="${prefix}link4_to_${prefix}link5" type="revolute">
+    <joint name="${prefix}link4_to_${prefix}link5" type="fixed">
       <axis xyz="0 0 1"/>
       <limit effort="${joint_effort}" lower="-2.5830" upper="2.5830" velocity="${joint_velocity}"/>
